Commit message: no limits xacro file

File: gym-simulations/gym_simulations/render/two_panda_world_no_limits.xacro (robot description, xacro)
@@ -3,5 +3,5 @@
   <xacro:arg name="arm_id_1" default="panda_0" />
   <xacro:arg name="arm_id_2" default="panda_1" />
-  <xacro:include filename="$(find franka_description)/robots/panda_arm.xacro"/>
+  <xacro:include filename="$(find franka_description)/robots/panda_arm_no_limits.xacro"/>
   <xacro:include filename="$(find franka_description)/robots/hand.xacro"/>
   <!-- box shaped table as base for the 2 Pandas -->
@@ -13,5 +13,5 @@
       </geometry>
       <material name="Tan">
-        <color rgba=".7 .7 .4 1.0"/>
+        <color rgba=".4 .9 .4 1.0"/>
       </material>
     </visual>
@@ -35,8 +35,8 @@
       <origin xyz="0 0 0." rpy="0 0 0"/>
       <geometry>
-        <cylinder length=".015" radius=".04"/>
-      </geometry>
-      <material name="blue">
-        <color rgba=".2 .6 .9 1.0"/>
+        <cylinder length=".03" radius=".04"/>
+      </geometry>
+      <material name="blue">
+        <color rgba=".15 .5 .7 1.0"/>
       </material>
     </visual>
@@ -50,8 +50,8 @@
       <origin xyz="0 0 0." rpy="0 0 0"/>
       <geometry>
-        <cylinder length=".015" radius=".04"/>
-      </geometry>
-      <material name="blue">
-        <color rgba=".2 .6 .9 1.0"/>
+        <cylinder length=".03" radius=".04"/>
+      </geometry>
+      <material name="blue">
+        <color rgba=".15 .5 .7 1.0"/>
       </material>
     </visual>
@@ -65,8 +65,8 @@
       <origin xyz="0 0 0." rpy="0 0 0"/>
       <geometry>
-        <cylinder length=".015" radius=".04"/>
-      </geometry>
-      <material name="blue">
-        <color rgba=".2 .6 .9 1.0"/>
+        <cylinder length=".03" radius=".04"/>
+      </geometry>
+      <material name="blue">
+        <color rgba=".15 .5 .7 1.0"/>
       </material>
     </visual>
@@ -80,8 +80,8 @@
       <origin xyz="0 0 0." rpy="0 0 0"/>
       <geometry>
-        <cylinder length=".015" radius=".04"/>
-      </geometry>
-      <material name="blue">
-        <color rgba=".2 .6 .9 1.0"/>
+        <cylinder length=".03" radius=".04"/>
+      </geometry>
+      <material name="blue">
+        <color rgba=".15 .5 .7 1.0"/>
       </material>
     </visual>
@@ -95,8 +95,8 @@
       <origin xyz="0 0 0." rpy="0 0 0"/>
       <geometry>
-        <cylinder length=".015" radius=".04"/>
-      </geometry>
-      <material name="blue">
-        <color rgba=".2 .6 .9 1.0"/>
+        <cylinder length=".03" radius=".04"/>
+      </geometry>
+      <material name="blue">
+        <color rgba=".15 .5 .7 1.0"/>
       </material>
     </visual>
@@ -111,8 +111,8 @@
       <origin xyz="0 0 0." rpy="0 0 0"/>
       <geometry>
-        <cylinder length=".015" radius=".04"/>
-      </geometry>
-      <material name="red">
-        <color rgba="1. .4 .1 1.0"/>
+        <cylinder length=".03" radius=".04"/>
+      </geometry>
+      <material name="red">
+        <color rgba=".7 .1 .1 1.0"/>
       </material>
     </visual>
@@ -126,8 +126,8 @@
       <origin xyz="0 0 0." rpy="0 0 0"/>
       <geometry>
-        <cylinder length=".015" radius=".04"/>
-      </geometry>
-      <material name="red">
-        <color rgba="1. .4 .1 1.0"/>
+        <cylinder length=".03" radius=".04"/>
+      </geometry>
+      <material name="red">
+        <color rgba=".7 .1 .1 1.0"/>
       </material>
     </visual>
@@ -141,8 +141,8 @@
       <origin xyz="0 0 0." rpy="0 0 0"/>
       <geometry>
-        <cylinder length=".015" radius=".04"/>
-      </geometry>
-      <material name="red">
-        <color rgba="1. .4 .1 1.0"/>
+        <cylinder length=".03" radius=".04"/>
+      </geometry>
+      <material name="red">
+        <color rgba=".7 .1 .1 1.0"/>
       </material>
     </visual>
@@ -156,8 +156,8 @@
       <origin xyz="0 0 0." rpy="0 0 0"/>
       <geometry>
-        <cylinder length=".015" radius=".04"/>
-      </geometry>
-      <material name="red">
-        <color rgba="1. .4 .1 1.0"/>
+        <cylinder length=".03" radius=".04"/>
+      </geometry>
+      <material name="red">
+        <color rgba=".7 .1 .1 1.0"/>
       </material>
     </visual>
@@ -171,8 +171,8 @@
       <origin xyz="0 0 0." rpy="0 0 0"/>
       <geometry>
-        <cylinder length=".015" radius=".04"/>
-      </geometry>
-      <material name="red">
-        <color rgba="1. .4 .1 1.0"/>
+        <cylinder length=".03" radius=".04"/>
+      </geometry>
+      <material name="red">
+        <color rgba=".7 .1 .1 1.0"/>
       </material>
     </visual>
@@ -182,3 +182,36 @@
     <child link="red_tok_4"/>
   </joint>
+  <!-- Bins -->
+  <!-- Blue -->
+  <link name="blue_bin">
+    <visual>
+      <origin xyz="0 0 0." rpy="0 0 0"/>
+      <geometry>
+        <cylinder length=".015" radius=".30"/>
+      </geometry>
+      <material name="light blue">
+        <color rgba="0.2 .5 1 1.0"/>
+      </material>
+    </visual>
+  </link>
+  <joint name="blue_bin_link" type="floating">
+    <parent link="base"/>
+    <child link="blue_bin"/>
+  </joint>
+  <!-- Red -->
+  <link name="red_bin">
+    <visual>
+      <origin xyz="0 0 0." rpy="0 0 0"/>
+      <geometry>
+        <cylinder length=".015" radius=".30"/>
+      </geometry>
+      <material name="light red">
+        <color rgba="1 .2 .3 1.0"/>
+      </material>
+    </visual>
+  </link>
+  <joint name="red_bin_link" type="floating">
+    <parent link="base"/>
+    <child link="red_bin"/>
+  </joint>
 </robot>
